Commit message: dialing in

File: src/jax_description/urdf/jax.urdf (robot description, URDF)
Before this commit: robot jax, 17 links, 16 joints
Links:
- link FL_link4: geometry collision sphere radius=0.009; visual mesh filename=package://jax_description/meshes/link4.dae
- link FR_link4: geometry collision sphere radius=0.009; visual mesh filename=package://jax_description/meshes/link4.dae
- link RL_link4: geometry collision sphere radius=0.009; visual mesh filename=package://jax_description/meshes/link4.dae
- link RR_link4: geometry collision sphere radius=0.009; visual mesh filename=package://jax_description/meshes/link4.dae
